Commit message: commit 3

File: Kitcat/src/legged_examples/legged_dm_description/urdf/dm.urdf (robot description, URDF)
Before this commit: robot legged_dm_description_no_arm, 17 links, 16 joints
Links:
- link leg_l1_link: mass 0.48644139  -> 0.48644139
- link leg_l2_link: mass 0.11861238  -> 0.11861238
- link leg_l3_link: mass 0.96637716  -> 0.96637716
- link leg_l4_link: mass 0.59597545  -> 0.59597545
- link leg_l5_link: mass 0.15464822  -> 0.15464822
- link leg_r1_link: mass 0.48644139   -> 0.48644139
- link leg_r2_link: mass 0.11861238  -> 0.11861238
- link leg_r3_link: mass 0.96637716  -> 0.96637716
- link leg_r4_link: mass 0.59597545  -> 0.59597545
- link leg_r5_link: mass 0.15464822  -> 0.15464822
- link loin_yaw_Link: mass 1.24596075  -> 1.24596075
