Commit message: commit 2

File: Jet_HR2dot5/src/legged_examples/legged_dm_description/urdf/dm.urdf (robot description, URDF)
Before this commit: robot legged_dm_description_no_arm, 17 links, 16 joints
Links:
- link base_link: mass 8.80159264  -> 8.80159264
- link leg_l1_link: mass 0.08223546   -> 0.08223546
- link leg_l2_link: mass 0.43655515   -> 0.43655515
- link leg_l3_link: mass 1.06377080   -> 1.06377080
- link leg_l4_link: mass 1.15073554   -> 1.15073554
- link leg_l5_link: mass 0.94676044   -> 0.94676044
- link leg_r1_link: mass 0.08223546    -> 0.08223546
- link leg_r2_link: mass 0.43655515   -> 0.43655515
- link leg_r3_link: mass 1.06377080   -> 1.06377080
- link leg_r4_link: mass 1.15073554   -> 1.15073554
- link leg_r5_link: mass 0.94676044   -> 0.94676044
- link loin_yaw_Link: mass 1.65580951   -> 1.65580951
Joints:
- joint leg_l5_fixed_1: origin xyz=0.113 -0.008 -0.006 rpy=0 0 0 -> xyz=0.0954425 -0.026875 -0.1538 rpy=0 0 0
- joint leg_l5_fixed_2: origin xyz=-0.061 -0.008 -0.006 rpy=0 0 0 -> xyz=-0.12 -0.026875 -0.1538 rpy=0 0 0
- joint leg_r5_fixed_1: origin xyz=0.113 0.008 -0.006 rpy=0 0 0 -> xyz=0.0954425 0.026875 -0.1538 rpy=0 0 0
- joint leg_r5_fixed_2: origin xyz=-0.061 0.008 -0.006 rpy=0 0 0 -> xyz=-0.12 0.026875 -0.1538 rpy=0 0 0

Commit message: commit 3

File: Jet_HR2dot5/src/legged_examples/legged_dm_description/urdf/dm.urdf (robot description, URDF)
Before this commit: robot legged_dm_description_no_arm, 17 links, 16 joints
Joints:
- joint leg_l2_joint: limit lower=-1.05 upper=1.05 effort=52 velocity=20 -> lower=-0.52 upper=0.785 effort=52 velocity=20
- joint leg_l3_joint: limit lower=-0.52 upper=0.785 effort=52 velocity=20 -> lower=-1.57 upper=1.57 effort=52 velocity=20
- joint leg_l5_joint: limit lower=-1.047 upper=0.3 effort=52 velocity=20 -> lower=-1.57 upper=0.3 effort=52 velocity=20
- joint leg_r2_joint: limit lower=-1.05 upper=1.05 effort=52 velocity=20 -> lower=-0.785 upper=0.52 effort=52 velocity=20
- joint leg_r3_joint: limit lower=-0.785 upper=0.52 effort=52 velocity=20 -> lower=-1.57 upper=1.57 effort=52 velocity=20
- joint leg_r5_joint: limit lower=-1.047 upper=0.3 effort=52 velocity=20 -> lower=-1.57 upper=0.3 effort=52 velocity=20
